File: barduino.brd (EAGLE design)
At the start: 107.4 x 50.9 mm, 18 parts, among them Q2 16MHz, X1 MINI-USB-UX60A-MB-5ST

Commit message: lots of routing
Parts:
- moved SG1 25.2 mm to (-5.99, 43.5)
- moved C2 23.7 mm to (28.5, 34.7)
- moved S0 18.9 mm to (33.8, 47.8)
- moved S1 18.4 mm to (25.2, 47.8)
- moved X1 12.4 mm to (28.7, 13.0)
- moved ICSP 9.17 mm to (28.5, 27.3)
- moved R3 6.44 mm to (8.83, 47.9)
- moved C6 2.98 mm to (0.48, 32.0)
- moved C5 1.89 mm to (-3.91, 24.1)
- moved C4 1.22 mm to (-3.82, 29.2)
- moved C7 0.99 mm to (19.7, 28.4), turned to 270 degrees
- moved Q2 0.36 mm to (0.41, 24.7)
Connections:
- removed net N$3: R6.1, R6.2
- net SCK-D13: no longer R2.1, R2.2
- net VCC: no longer R7.1, R7.2
Routing:
- net GND: track 11.7 -> 94.8 mm
- net RESET: track 0.00 -> 66.4 mm
- net VCC: track 8.94 -> 50.5 mm
- net A0: track 0.00 -> 22.0 mm
- net A1: track 0.00 -> 16.1 mm
- net PB7: track 0.00 -> 12.0 mm
- net PB6: track 0.00 -> 10.7 mm
- net D10: track 0.00 -> 9.36 mm
- net D6: track 0.00 -> 7.53 mm
- net D5: track 0.00 -> 7.46 mm
- net A2: track 0.00 -> 7.43 mm
- net D2: track 0.00 -> 7.34 mm
- net D9: track 0.00 -> 6.96 mm
- net A3: track 0.00 -> 6.30 mm
- net D1: track 0.00 -> 6.30 mm
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
Commit message: some changes before moving the USB conn
Parts:
- moved R6 7.22 mm to (47.6, 23.7), turned to 180 degrees
- moved R2 2.90 mm to (46.3, 28.8)
- turned R7 to 180 degrees
Routing:
- net D3: track 0.00 -> 21.4 mm
- net SCK-D13: track 0.00 -> 15.2 mm
- net MISO-D12: track 0.09 -> 12.4 mm
- net RESET: track 66.4 -> 54.2 mm
- net VCC: track 50.5 -> 43.2 mm
- net GND: track 94.8 -> 89.2 mm
Changed lines of the file:
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@@
 <element name="U$1" library="fab" package="TQFP32-08THIN" value="ATMEGA88-THIN" x="10.8103" y="29.0983"/>
 <element name="ICSP" library="fab" package="2X03SMD" value="" x="28.514096875" y="27.335546875" rot="R90"/>
-<element name="R6" library="ng" package="1206" value="0" x="43.42644375" y="17.78514375" rot="R90"/>
-<element name="R7" library="ng" package="1206" value="0" x="49.268440625" y="18.1509" rot="R90"/>
-<element name="R2" library="ng" package="1206" value="0" x="46.7894" y="25.89028125" rot="R180"/>
+<element name="R6" library="ng" package="1206" value="0" x="47.617446875" y="23.660165625" rot="R180"/>
+<element name="R7" library="ng" package="1206" value="0" x="49.268440625" y="18.1509" rot="R180"/>
+<element name="R2" library="ng" package="1206" value="0" x="46.3042625" y="28.75031875" rot="R180"/>
 <element name="SG1" library="buzzer" library_urn="urn:adsk.eagle:library:113" package="F/CM12P" value="F/CM12P" x="-5.989321875" y="43.5432125" rot="R90">
 <attribute name="MF" value="" x="-5.989321875" y="43.5432125" size="1.778" layer="27" rot="R90" display="off"/>
@@
 <wire x1="21.346159375" y1="27.051" x2="19.66000625" y2="27.051" width="0.4064" layer="1"/>
 <wire x1="19.66000625" y1="27.051" x2="19.61270625" y2="27.0983" width="0.4064" layer="1"/>
-<wire x1="27.135021875" y1="15.2776625" x2="27.135021875" y2="16.634259375" width="0.4064" layer="1"/>
-<wire x1="27.135021875" y1="16.634259375" x2="19.712940625" y2="24.056340625" width="0.4064" layer="1"/>
-<wire x1="19.712940625" y1="24.056340625" x2="19.712940625" y2="26.998065625" width="0.4064" layer="1"/>
-<wire x1="19.712940625" y1="26.998065625" x2="19.705265625" y2="27.005740625" width="0.4064" layer="1"/>
-<wire x1="0.4826625" y1="30.627778125" x2="7.404440625" y2="47.919625" width="0" layer="19" extent="1-1"/>
+<wire x1="27.06878125" y1="16.79448125" x2="27.06878125" y2="15.343903125" width="0.4064" layer="1"/>
+<wire x1="27.06878125" y1="15.343903125" x2="27.075421875" y2="15.3372625" width="0.4064" layer="1"/>
+<wire x1="21.346159375" y1="27.051" x2="21.346159375" y2="17.58188125" width="0" layer="19" extent="1-16"/>
+<wire x1="21.346159375" y1="17.58188125" x2="22.01418125" y2="16.913859375" width="0.4064" layer="1"/>
+<wire x1="22.01418125" y1="16.913859375" x2="26.949403125" y2="16.913859375" width="0.4064" layer="1"/>
+<wire x1="26.949403125" y1="16.913859375" x2="27.06878125" y2="16.79448125" width="0.4064" layer="1"/>
+<wire x1="6.5177" y1="29.4983" x2="7.404440625" y2="47.919625" width="0" layer="19" extent="1-1"/>
+<wire x1="27.135021875" y1="15.2776625" x2="27.06878125" y2="15.343903125" width="0" layer="19" extent="1-1"/>
 </signal>
 <signal name="GND" class="1">
@@
 <wire x1="-3.9115375" y1="25.521578125" x2="-4.871378125" y2="25.521578125" width="0.4064" layer="1"/>
 <wire x1="-4.871378125" y1="25.521578125" x2="-5.946140625" y2="26.596340625" width="0.4064" layer="1"/>
-<wire x1="-5.946140625" y1="26.596340625" x2="-5.946140625" y2="30.020259375" width="0.4064" layer="1"/>
+<wire x1="-5.946140625" y1="29.657040625" x2="-5.946140625" y2="26.596340625" width="0.4064" layer="1"/>
+<wire x1="-5.946140625" y1="29.657040625" x2="-5.946140625" y2="30.020259375" width="0.4064" layer="1"/>
 <wire x1="-5.946140625" y1="30.020259375" x2="-5.344159375" y2="30.622240625" width="0.4064" layer="1"/>
 <wire x1="-3.856003125" y1="30.622240625" x2="-5.344159375" y2="30.622240625" width="0.4064" layer="1"/>
@@
 <wire x1="29.94151875" y1="36.210240625" x2="29.94151875" y2="34.7265" width="0.4064" layer="1"/>
 <wire x1="29.94151875" y1="34.7265" x2="29.953934375" y2="34.714084375" width="0.4064" layer="1"/>
-<wire x1="30.335021875" y1="15.2776625" x2="30.335021875" y2="22.184559375" width="0.4064" layer="1"/>
-<wire x1="30.335021875" y1="22.184559375" x2="29.82468125" y2="22.6949" width="0.4064" layer="1"/>
-<wire x1="29.82468125" y1="22.6949" x2="29.82468125" y2="23.25785625" width="0.4064" layer="1"/>
-<wire x1="29.82468125" y1="23.25785625" x2="29.809496875" y2="23.273040625" width="0.4064" layer="1"/>
-<wire x1="29.809496875" y1="23.273040625" x2="29.809496875" y2="26.7640375" width="0.4064" layer="1"/>
-<wire x1="29.809496875" y1="26.7640375" x2="30.914340625" y2="27.86888125" width="0.4064" layer="1"/>
-<wire x1="30.914340625" y1="27.86888125" x2="30.914340625" y2="30.115790625" width="0.4064" layer="1"/>
-<wire x1="30.914340625" y1="30.115790625" x2="31.054096875" y2="30.255546875" width="0.4064" layer="1"/>
 <wire x1="27.467559375" y1="44.460159375" x2="27.480259375" y2="44.460159375" width="0.4064" layer="1"/>
 <wire x1="27.480259375" y1="44.460159375" x2="29.664659375" y2="46.644559375" width="0.4064" layer="1"/>
@@
 <wire x1="36.062978125" y1="44.452603125" x2="36.062978125" y2="42.3317" width="0.4064" layer="1"/>
 <wire x1="36.062978125" y1="42.3317" x2="29.94151875" y2="36.210240625" width="0.4064" layer="1"/>
-<wire x1="-5.989321875" y1="39.7332125" x2="-5.946140625" y2="26.596340625" width="0" layer="19" extent="1-1"/>
+<wire x1="-5.989321875" y1="39.7332125" x2="-5.989321875" y2="29.700221875" width="0.4064" layer="1"/>
+<wire x1="-5.989321875" y1="29.700221875" x2="-5.946140625" y2="29.657040625" width="0.4064" layer="1"/>
+<wire x1="31.054096875" y1="30.255546875" x2="30.335021875" y2="15.2776625" width="0" layer="19" extent="1-1"/>
 </signal>
 <signal name="PB7">
@@
 <contactref element="U$1" pad="29"/>
 <contactref element="ICSP" pad="5"/>
-<wire x1="31.054096875" y1="24.795546875" x2="31.054096875" y2="26.859153125" width="0.4064" layer="1"/>
-<wire x1="31.054096875" y1="26.859153125" x2="32.298696875" y2="28.103753125" width="0.4064" layer="1"/>
+<wire x1="31.054096875" y1="24.795546875" x2="31.054096875" y2="26.859153125" width="0" layer="19" extent="1-16"/>
+<wire x1="31.054096875" y1="26.859153125" x2="32.298696875" y2="28.103753125" width="0" layer="19" extent="1-16"/>
 <wire x1="32.298696875" y1="36.459215625" x2="35.814" y2="39.97451875" width="0.4064" layer="1"/>
-<wire x1="32.298696875" y1="28.103753125" x2="32.298696875" y2="36.459215625" width="0.4064" layer="1"/>
+<wire x1="32.298696875" y1="28.103753125" x2="32.298696875" y2="36.459215625" width="0" layer="19" extent="1-16"/>
 <wire x1="37.434578125" y1="45.848109375" x2="37.077484375" y2="46.205203125" width="0.4064" layer="1"/>
 <wire x1="37.077484375" y1="46.205203125" x2="36.819778125" y2="46.205203125" width="0.4064" layer="1"/>
@@
 <contactref element="U$1" pad="17"/>
 <contactref element="ICSP" pad="3"/>
-<wire x1="15.1791" y1="26.2983" x2="28.514096875" y2="24.795546875" width="0" layer="19" extent="1-1"/>
+<wire x1="15.1791" y1="26.2983" x2="17.25761875" y2="26.2983" width="0.4064" layer="1"/>
+<wire x1="17.25761875" y1="26.2983" x2="18.16861875" y2="25.3873" width="0.4064" layer="1"/>
+<wire x1="18.16861875" y1="25.3873" x2="23.79874375" y2="25.3873" width="0.4064" layer="1"/>
+<wire x1="23.79874375" y1="25.3873" x2="25.086590625" y2="26.675146875" width="0.4064" layer="1"/>
+<wire x1="26.861603125" y1="26.675146875" x2="27.218696875" y2="26.318053125" width="0.4064" layer="1"/>
+<wire x1="27.218696875" y1="26.318053125" x2="27.218696875" y2="26.090946875" width="0.4064" layer="1"/>
+<wire x1="27.218696875" y1="26.090946875" x2="28.514096875" y2="24.795546875" width="0.4064" layer="1"/>
+<wire x1="25.086590625" y1="26.675146875" x2="26.861603125" y2="26.675146875" width="0.4064" layer="1"/>
 </signal>
 <signal name="A0">
@@
 <contactref element="U$1" pad="1"/>
 <contactref element="SG1" pad="+"/>
-<wire x1="-5.989321875" y1="47.3532125" x2="6.4415" y2="31.8983" width="0" layer="19" extent="1-1"/>
+<wire x1="6.4415" y1="31.8983" x2="5.1069625" y2="31.8983" width="0.4064" layer="1"/>
+<wire x1="5.1069625" y1="31.8983" x2="-0.36321875" y2="37.36848125" width="0.4064" layer="1"/>
+<wire x1="-0.36321875" y1="37.36848125" x2="-0.36321875" y2="41.727109375" width="0.4064" layer="1"/>
+<wire x1="-0.36321875" y1="41.727109375" x2="-5.989321875" y2="47.3532125" width="0.4064" layer="1"/>
 </signal>
 <signal name="D4">
@@
 <contactref element="U$1" pad="16"/>
 <contactref element="ICSP" pad="1"/>
-<wire x1="13.6103" y1="24.7295" x2="25.90805" y2="24.7295" width="0" layer="19" extent="1-16"/>
 <wire x1="25.90805" y1="24.7295" x2="25.974096875" y2="24.795546875" width="0.4064" layer="1"/>
+<wire x1="13.6103" y1="24.7295" x2="25.90805" y2="24.7295" width="0.4064" layer="1"/>
 </signal>
 <signal name="N$6">

Commit message: USB move is going well
Parts:
- removed C6: .1uF, ng:1206
- removed R6, R7: 0, ng:1206
- moved X1 51.6 mm to (-19.9, 30.3), turned to 0 degrees
- moved R2 43.9 mm to (2.41, 28.7), turned to 90 degrees
- moved C4 5.43 mm to (-6.47, 24.4), turned to 0 degrees
- moved C5 4.94 mm to (-6.49, 19.9), turned to 0 degrees
- moved Q2 3.00 mm to (-1.19, 22.2)
Connections:
- new net N$2: R2.2, X1.1
- net GND: no longer C6.1
- net VCC: now also R2.1; no longer C6.2, X1.1
Routing:
- net MOSI-D11: track 2.20 -> 27.7 mm
- net N$2: track 0.00 -> 20.8 mm
- net VCC: track 43.2 -> 25.8 mm
- net RESET: track 54.2 -> 66.4 mm
- net PB7: track 12.0 -> 14.8 mm
- net PB6: track 10.7 -> 12.7 mm
- net GND: track 89.2 -> 88.3 mm

Commit message: board fully laid out
Parts:
- ICSP: value (none) -> PROG
- S0: value (none) -> HR
- S1: value (none) -> MIN
Connections:
- removed net N$2: R2.2, X1.1
- new net VUSB: R2.2, R3.2, X1.1
- net VCC: no longer R3.2
Routing:
- net VUSB: track 0.00 -> 55.7 mm
- net N$2: track 20.8 -> 0.00 mm
- net GND: track 88.3 -> 107.5 mm
- net VCC: track 25.8 -> 34.8 mm
- net N$18: track 1.84 -> 0.00 mm
- net N$17: track 1.39 -> 0.00 mm
Other:
- board size 107.4 x 50.9 mm -> 68.5 x 37.2 mm

Commit message: remove crossover resistor
Parts:
- removed R2: 0, ng:1206
- moved X1 3.64 mm to (-16.3, 30.3)
Connections:
- removed net VUSB: R2.2, R3.2, X1.1
- net VCC: now also R3.2, X1.1; no longer R2.1
Routing:
- net VCC: track 34.8 -> 133.1 mm
- net VUSB: track 55.7 -> 0.00 mm
- net GND: track 107.5 -> 103.0 mm
Changed lines of the file:
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@@
 <element name="U$1" library="fab" package="TQFP32-08THIN" value="ATMEGA88-THIN" x="10.8103" y="29.0983"/>
 <element name="ICSP" library="fab" package="2X03SMD" value="PROG" x="28.514096875" y="27.335546875" rot="R90"/>
-<element name="R2" library="ng" package="1206" value="0" x="2.40544375" y="28.71221875" rot="R90"/>
 <element name="SG1" library="buzzer" library_urn="urn:adsk.eagle:library:113" package="F/CM12P" value="F/CM12P" x="-5.989321875" y="43.5432125" rot="R90">
 <attribute name="MF" value="" x="-5.989321875" y="43.5432125" size="1.778" layer="27" rot="R90" display="off"/>
@@
 <attribute name="OC_NEWARK" value="unknown" x="-5.989321875" y="43.5432125" size="1.778" layer="27" rot="R90" display="off"/>
 </element>
-<element name="X1" library="con-hirose" library_urn="urn:adsk.eagle:library:152" package="UX60A-MB-5ST" value="MINI-USB-UX60A-MB-5ST" x="-19.933915625" y="30.31998125">
-<attribute name="MF" value="" x="-19.933915625" y="30.31998125" size="1.778" layer="27" display="off"/>
-<attribute name="MPN" value="" x="-19.933915625" y="30.31998125" size="1.778" layer="27" display="off"/>
-<attribute name="OC_FARNELL" value="unknown" x="-19.933915625" y="30.31998125" size="1.778" layer="27" display="off"/>
-<attribute name="OC_NEWARK" value="unknown" x="-19.933915625" y="30.31998125" size="1.778" layer="27" display="off"/>
+<element name="X1" library="con-hirose" library_urn="urn:adsk.eagle:library:152" package="UX60A-MB-5ST" value="MINI-USB-UX60A-MB-5ST" x="-16.289015625" y="30.31998125">
+<attribute name="MF" value="" x="-16.289015625" y="30.31998125" size="1.778" layer="27" display="off"/>
+<attribute name="MPN" value="" x="-16.289015625" y="30.31998125" size="1.778" layer="27" display="off"/>
+<attribute name="OC_FARNELL" value="unknown" x="-16.289015625" y="30.31998125" size="1.778" layer="27" display="off"/>
+<attribute name="OC_NEWARK" value="unknown" x="-16.289015625" y="30.31998125" size="1.778" layer="27" display="off"/>
 </element>
 <element name="S1" library="ng" package="6MM_SWITCH" value="MIN" x="25.181559375" y="47.762159375" rot="R90"/>
@@
 <wire x1="25.974096875" y1="30.255546875" x2="25.974096875" y2="33.578246875" width="0.4064" layer="1"/>
 <wire x1="25.974096875" y1="33.578246875" x2="27.109934375" y2="34.714084375" width="0.4064" layer="1"/>
-<contactref element="R2" pad="1"/>
 <contactref element="C7" pad="2"/>
 <contactref element="U$1" pad="6"/>
@@
 <wire x1="9.244540625" y1="27.8983" x2="9.922509375" y2="28.57626875" width="0.4064" layer="1"/>
 <wire x1="4.220421875" y1="27.8983" x2="6.5177" y2="27.8983" width="0.4064" layer="1"/>
-<wire x1="2.40544375" y1="27.29021875" x2="3.612340625" y2="27.29021875" width="0.4064" layer="1"/>
-<wire x1="3.612340625" y1="27.29021875" x2="4.220421875" y2="27.8983" width="0.4064" layer="1"/>
+<contactref element="X1" pad="1"/>
+<wire x1="-14.039015625" y1="31.91998125" x2="-13.111678125" y2="31.91998125" width="0.4064" layer="1"/>
+<wire x1="-13.111678125" y1="31.91998125" x2="-12.065" y2="32.966659375" width="0.4064" layer="1"/>
+<wire x1="-12.065" y1="36.86048125" x2="-12.065" y2="32.966659375" width="0.4064" layer="1"/>
+<wire x1="-12.065" y1="36.86048125" x2="-20.460621875" y2="36.86048125" width="0.4064" layer="1"/>
+<wire x1="-20.460621875" y1="36.86048125" x2="-22.892215625" y2="34.4288875" width="0.4064" layer="1"/>
+<wire x1="-9.3187" y1="18.72916875" x2="-8.96160625" y2="18.372075" width="0.4064" layer="1"/>
+<wire x1="-8.96160625" y1="18.372075" x2="-6.85659375" y2="18.372075" width="0.4064" layer="1"/>
+<wire x1="-6.608340625" y1="27.8855" x2="-6.273253125" y2="27.88484375" width="0.4064" layer="1"/>
+<wire x1="-6.273253125" y1="27.88484375" x2="-6.27259375" y2="27.8855" width="0.4064" layer="1"/>
+<wire x1="-6.27259375" y1="27.8855" x2="4.220421875" y2="27.8855" width="0.4064" layer="1"/>
+<wire x1="-6.4868" y1="27.763959375" x2="-6.608340625" y2="27.8855" width="0.4064" layer="1"/>
+<wire x1="-22.892215625" y1="26.211075" x2="-20.941521875" y2="24.26038125" width="0.4064" layer="1"/>
+<wire x1="-6.85659375" y1="18.372075" x2="-6.4868" y2="18.74186875" width="0.4064" layer="1"/>
+<wire x1="-6.4868" y1="18.74186875" x2="-6.4868" y2="27.763959375" width="0.4064" layer="1"/>
+<wire x1="-20.941521875" y1="24.26038125" x2="-9.3187" y2="24.237621875" width="0.4064" layer="1"/>
+<wire x1="-9.3187" y1="24.237621875" x2="-9.3187" y2="18.72916875" width="0.4064" layer="1"/>
+<wire x1="-22.892215625" y1="34.4288875" x2="-22.892215625" y2="26.211075" width="0.4064" layer="1"/>
+<contactref element="R3" pad="2"/>
+<wire x1="7.404440625" y1="47.919625" x2="-2.646665625" y2="47.919625" width="0.4064" layer="1"/>
+<wire x1="-2.646665625" y1="47.919625" x2="-3.959859375" y2="49.23281875" width="0.4064" layer="1"/>
+<wire x1="-3.959859375" y1="49.23281875" x2="-5.2107625" y2="49.23281875" width="0.4064" layer="1"/>
+<wire x1="-5.2107625" y1="49.23281875" x2="-5.210765625" y2="49.232821875" width="0.4064" layer="1"/>
+<wire x1="-5.210765625" y1="49.232821875" x2="-9.050015625" y2="49.232821875" width="0.4064" layer="1"/>
+<wire x1="-9.050015625" y1="49.232821875" x2="-10.024109375" y2="48.258728125" width="0.4064" layer="1"/>
+<wire x1="-10.024109375" y1="48.258728125" x2="-10.18031875" y2="48.10251875" width="0.4064" layer="1"/>
+<wire x1="-10.18031875" y1="48.10251875" x2="-10.1117375" y2="48.10251875" width="0.4064" layer="1"/>
+<wire x1="-10.024109375" y1="48.258728125" x2="-10.024109375" y2="38.901371875" width="0.4064" layer="1"/>
+<wire x1="-10.024109375" y1="38.901371875" x2="-12.065" y2="36.86048125" width="0.4064" layer="1"/>
+<wire x1="4.220421875" y1="27.8855" x2="4.220421875" y2="27.8983" width="0" layer="19" extent="1-1"/>
 </signal>
 <signal name="GND" class="1">
@@
 <wire x1="36.062978125" y1="42.3317" x2="29.94151875" y2="36.210240625" width="0.4064" layer="1"/>
 <wire x1="-6.6083375" y1="28.6983" x2="-8.17528125" y2="28.70136875" width="0.4064" layer="1"/>
-<wire x1="-10.304521875" y1="28.7055375" x2="-8.17528125" y2="28.70136875" width="0.4064" layer="1"/>
-<wire x1="-10.304521875" y1="28.7055375" x2="-17.683915625" y2="28.71998125" width="0.4064" layer="1"/>
+<wire x1="-8.17528125" y1="28.70136875" x2="-10.304521875" y2="28.7055375" width="0.4064" layer="1"/>
 <wire x1="-7.9091" y1="19.883175" x2="-7.9091" y2="24.41708125" width="0.4064" layer="1"/>
 <wire x1="-7.9091" y1="24.41708125" x2="-7.8964" y2="24.42978125" width="0.4064" layer="1"/>
@@
 <wire x1="3.55945" y1="31.54381875" x2="2.200071875" y2="31.54381875" width="0.4064" layer="1"/>
 <wire x1="2.200071875" y1="31.54381875" x2="-5.989321875" y2="39.7332125" width="0.4064" layer="1"/>
-<wire x1="4.64058125" y1="28.71110625" x2="4.64058125" y2="30.4626875" width="0.4064" layer="1"/>
+<wire x1="4.64058125" y1="29.6164" x2="4.64058125" y2="30.4626875" width="0.4064" layer="1"/>
 <wire x1="4.64058125" y1="30.4626875" x2="3.55945" y2="31.54381875" width="0.4064" layer="1"/>
+<wire x1="-10.304521875" y1="28.7055375" x2="-12.741353125" y2="28.7055375" width="0.4064" layer="1"/>
+<wire x1="-12.741353125" y1="28.7055375" x2="-12.786509375" y2="28.66038125" width="0.4064" layer="1"/>
+<wire x1="-12.786509375" y1="28.66038125" x2="-14.039015625" y2="28.66038125" width="0.4064" layer="1"/>
 <wire x1="6.5177" y1="28.6983" x2="6.5177" y2="30.2983" width="0" layer="19" extent="1-1"/>
+<wire x1="-14.039015625" y1="28.71998125" x2="-14.039015625" y2="28.66038125" width="0" layer="19" extent="1-1"/>
 </signal>
 <signal name="PB7">
@@
 <wire x1="12.0852" y1="26.2738" x2="12.0675" y2="26.2915" width="0.4064" layer="1"/>
 </signal>
-<signal name="VUSB" class="1">
-<contactref element="R2" pad="2"/>
-<contactref element="X1" pad="1"/>
-<contactref element="R3" pad="2"/>
-<wire x1="7.404440625" y1="47.919625" x2="-2.646665625" y2="47.919625" width="0.4064" layer="1"/>
-<wire x1="-2.646665625" y1="47.919625" x2="-3.959859375" y2="49.23281875" width="0.4064" layer="1"/>
-<wire x1="-3.959859375" y1="49.23281875" x2="-5.2107625" y2="49.23281875" width="0.4064" layer="1"/>
-<wire x1="-5.2107625" y1="49.23281875" x2="-5.210765625" y2="49.232821875" width="0.4064" layer="1"/>
-<wire x1="-5.210765625" y1="49.232821875" x2="-9.050015625" y2="49.232821875" width="0.4064" layer="1"/>
-<wire x1="-9.050015625" y1="49.232821875" x2="-10.18031875" y2="48.10251875" width="0.4064" layer="1"/>
-<wire x1="-10.18031875" y1="48.10251875" x2="-10.1117375" y2="48.10251875" width="0.4064" layer="1"/>
-<wire x1="-10.132059375" y1="31.91998125" x2="-17.683915625" y2="31.91998125" width="0.4064" layer="1"/>
-<wire x1="-10.132059375" y1="31.91998125" x2="0.61968125" y2="31.91998125" width="0.4064" layer="1"/>
-<wire x1="0.61968125" y1="31.91998125" x2="2.40544375" y2="30.13421875" width="0.4064" layer="1"/>
-<wire x1="-10.18031875" y1="48.10251875" x2="-10.18031875" y2="31.968240625" width="0.4064" layer="1"/>
-<wire x1="-10.18031875" y1="31.968240625" x2="-10.132059375" y2="31.91998125" width="0.4064" layer="1"/>
-</signal>
 </signals>
